File: ri3ka.kicad_sch (KiCad schematic)
At the start: 0 parts

Commit message: tmp
Parts:
- added C1, C10, C11: 10uF, Capacitor_SMD:C_0805_2012Metric_Pad1.18x1.45mm_HandSolder, symbol Device:C
- added C12, C13, C14, C16, C18, C19, C2, C20, C21, C22, C23, C24, C5: 100nF, Capacitor_SMD:C_0805_2012Metric_Pad1.18x1.45mm_HandSolder, symbol Device:C
- added C15, C17: 10nF, Capacitor_SMD:C_0805_2012Metric_Pad1.18x1.45mm_HandSolder, symbol Device:C
- added C25, C26, C27, C28: 300uF, Capacitor_SMD:CP_Elec_5x3, symbol Device:C_Polarized
- added C29: C, Capacitor_SMD:C_0805_2012Metric_Pad1.18x1.45mm_HandSolder, symbol Device:C
- added C3, C4: 2.2uF, Capacitor_SMD:C_0805_2012Metric_Pad1.18x1.45mm_HandSolder, symbol Device:C
- added C6: 39pF, Capacitor_SMD:C_0805_2012Metric_Pad1.18x1.45mm_HandSolder, symbol Device:C
- added C7: 6.8nF, Capacitor_SMD:C_0805_2012Metric_Pad1.18x1.45mm_HandSolder, symbol Device:C
- added C8, C9: 47uF, Capacitor_SMD:C_0805_2012Metric_Pad1.18x1.45mm_HandSolder, symbol Device:C
- added D1: B560C-13-F, lib:SMC, symbol B560C-13-F:B560C-13-F
- added D10, D11, D12, D2, D3, D4, D5, D6, D9: LED, LED_SMD:LED_1206_3216Metric_Pad1.42x1.75mm_HandSolder, symbol Device:LED
- added J1: Screw_Terminal_01x02, TerminalBlock_4Ucon:TerminalBlock_4Ucon_1x02_P3.50mm_Horizontal, symbol Connector:Screw_Terminal_01x02
- added J10, J11, J12, J9: Conn_01x02_Socket, Connector_JST:JST_PH_B2B-PH-K_1x02_P2.00mm_Vertical, symbol Connector:Conn_01x02_Socket
- added J13, J14, J15, J16: Conn_01x03_Pin, Connector_JST:JST_PH_B3B-PH-K_1x03_P2.00mm_Vertical, symbol Connector:Conn_01x03_Pin
- added J2: USB_C_Receptacle_USB2.0_14P, Connector_USB:USB_C_Receptacle_HRO_TYPE-C-31-M-12, symbol Connector:USB_C_Receptacle_USB2.0_14P
- added J3: MOT_XA, Connector_JST:JST_PH_B4B-PH-K_1x04_P2.00mm_Vertical, symbol Connector:Conn_01x04_Socket
- added J4: MOT_YA, Connector_JST:JST_PH_B4B-PH-K_1x04_P2.00mm_Vertical, symbol Connector:Conn_01x04_Socket
- added J5: MOT_Z, Connector_JST:JST_PH_B4B-PH-K_1x04_P2.00mm_Vertical, symbol Connector:Conn_01x04_Socket
- added J6: MOT_A, Connector_JST:JST_PH_B4B-PH-K_1x04_P2.00mm_Vertical, symbol Connector:Conn_01x04_Socket
- added J7: MOT_YB, Connector_JST:JST_PH_B4B-PH-K_1x04_P2.00mm_Vertical, symbol Connector:Conn_01x04_Socket
- added J8: MOT_XB, Connector_JST:JST_PH_B4B-PH-K_1x04_P2.00mm_Vertical, symbol Connector:Conn_01x04_Socket
- added L1: 10uH, Inductor_SMD:L_0805_2012Metric_Pad1.15x1.40mm_HandSolder, symbol Device:L
- added MICRO_SD1: TF-01A, TF-01A:TF-01A, symbol TF-01A:TF-01A
- added Q1: PMBT3904YS, Package_TO_SOT_SMD:SOT-363_SC-70-6_Handsoldering, symbol Transistor_BJT:PMBT3904YS
- added R1: 100k, Resistor_SMD:R_0805_2012Metric_Pad1.20x1.40mm_HandSolder, symbol Device:R
- added R10, R13, R14, R16, R31, R41, R43, R45, R47, R9: 1k, Resistor_SMD:R_0805_2012Metric_Pad1.20x1.40mm_HandSolder, symbol Device:R
- added R11, R12, R15, R17, R20, R21, R22, R23, R24, R25, R26, R32, R42, R44, R46, R48, R8: 10k, Resistor_SMD:R_0805_2012Metric_Pad1.20x1.40mm_HandSolder, symbol Device:R
- added R18, R19: 5.1k, Resistor_SMD:R_0805_2012Metric_Pad1.20x1.40mm_HandSolder, symbol Device:R
- added R2: 13k, Resistor_SMD:R_0805_2012Metric_Pad1.20x1.40mm_HandSolder, symbol Device:R
- added R27, R28, R29, R30, R37, R38, R39, R40, R5: 6.8k, Resistor_SMD:R_0805_2012Metric_Pad1.20x1.40mm_HandSolder, symbol Device:R
- added R3: 270k, Resistor_SMD:R_0805_2012Metric_Pad1.20x1.40mm_HandSolder, symbol Device:R
- added R33, R34, R35, R36: 300, Resistor_SMD:R_0805_2012Metric_Pad1.20x1.40mm_HandSolder, symbol Device:R
- added R4: 51k, Resistor_SMD:R_0805_2012Metric_Pad1.20x1.40mm_HandSolder, symbol Device:R
- added R6, R7: R, Resistor_SMD:R_0805_2012Metric_Pad1.20x1.40mm_HandSolder, symbol Device:R
- added SW1: Reset, Button_Switch_SMD:SW_SPST_CK_KMS2xxGP, symbol Switch:CK_KMS2xxGP
- added SW2: Boot, Button_Switch_SMD:SW_SPST_CK_KMS2xxGP, symbol Switch:CK_KMS2xxGP
- added U1: ESP32-WROOM-32E, RF_Module:ESP32-WROOM-32E, symbol RF_Module:ESP32-WROOM-32E
- added U10: DRV_Z, TMC2209:MODULE_TMC2209_SILENTSTEPSTICK, symbol TMC_SILENTSTEPSTIC:TMC5160_SILENTSTEPSTICK
- added U11: DRV_A, TMC2209:MODULE_TMC2209_SILENTSTEPSTICK, symbol TMC_SILENTSTEPSTIC:TMC5160_SILENTSTEPSTICK
- added U12: TLP521-4, Package_SO:SOIC-16_3.9x9.9mm_P1.27mm, symbol Isolator:PC847
- added U13: 74AHCT125, Package_SO:SOIC-14_3.9x8.7mm_P1.27mm, symbol 74xx:74AHCT125
- added U2: TPS54360DDA, Package_SO:TI_SO-PowerPAD-8_ThermalVias, symbol Regulator_Switching:TPS54360DDA
- added U3: AMS1117-3.3, Package_TO_SOT_SMD:SOT-223-3_TabPin2, symbol Regulator_Linear:AMS1117-3.3
- added U4: CP2102N-Axx-xQFN28, Package_DFN_QFN:QFN-28-1EP_5x5mm_P0.5mm_EP3.25x3.25mm, symbol Interface_USB:CP2102N-Axx-xQFN28
- added U5: TPD3E001DRLR, Package_TO_SOT_SMD:SOT-553, symbol Power_Protection:TPD3E001DRLR
- added U6, U7: 74AHCT595, Package_SO:SOIC-16W_5.3x10.2mm_P1.27mm, symbol 74xx:74AHCT595
- added U8: DRV_X, TMC2209:MODULE_TMC2209_SILENTSTEPSTICK, symbol TMC_SILENTSTEPSTIC:TMC5160_SILENTSTEPSTICK
- added U9: DRV_Y, TMC2209:MODULE_TMC2209_SILENTSTEPSTICK, symbol TMC_SILENTSTEPSTIC:TMC5160_SILENTSTEPSTICK
Connections:
- new net: D6.1 (K), R40.2
- new net: D6.2 (A), J12.2 (Pin_2)
- new net: R9.1, SW1.1
- new net: Q1.5 (B2), R7.2
- new net: J15.3 (Pin_3), U13.8
- new net: D11.2 (A), R29.2
- new net: C5.1, U2.1 (BOOT)
- new net: R1.1, U2.4 (RT/CLK)
- new net: R3.2, R4.1, U2.5 (FB)
- new net: C6.1, R2.1, U2.6 (COMP)
- new net: C5.2, D1.C, L1.1, U2.8 (SW)
- new net: J13.3 (Pin_3), U13.3
- new net: J16.3 (Pin_3), U13.11
- new net: J3.3 (Pin_3), J8.3 (Pin_3), U8.3 (M1B)
- new net: J3.1 (Pin_1), J8.2 (Pin_2), U8.4 (M1A)
- new net: J3.2 (Pin_2), J8.1 (Pin_1), U8.5 (M2A)
- new net: J3.4 (Pin_4), J8.4 (Pin_4), U8.6 (M2B)
- new net: R31.1, U12.10
- new net: R41.2, R42.2, U13.2
- new net: D3.1 (K), R37.2
- new net: D3.2 (A), J9.2 (Pin_2)
- new net: R16.1, U12.12
- new net: R35.2, U12.6
- new net: J10.1 (Pin_1), R34.1
- new net: R34.2, U12.4
- new net: Q1.2 (B1), R6.2
- new net: J11.1 (Pin_1), R35.1
- new net: D5.2 (A), J11.2 (Pin_2)
- new net: R13.1, U12.16
- new net: J5.3 (Pin_3), U10.3 (M1B)
- new net: J5.1 (Pin_1), U10.4 (M1A)
- new net: J5.2 (Pin_2), U10.5 (M2A)
- new net: J5.4 (Pin_4), U10.6 (M2B)
- new net: D10.2 (A), R28.2
- new net: R47.2, R48.2, U13.12
- new net: D5.1 (K), R39.2
- new net: J2.A6 (D+), J2.B6 (D+), U4.4 (D+), U5.2 (IO2)
- new net: J2.A7 (D-), J2.B7 (D-), U4.5 (D-), U5.1 (IO1)
- new net: R43.2, R44.2, U13.5
- new net: C7.1, R2.2
- new net: J4.3 (Pin_3), J7.3 (Pin_3), U9.3 (M1B)
- new net: J4.1 (Pin_1), J7.2 (Pin_2), U9.4 (M1A)
- new net: J4.2 (Pin_2), J7.1 (Pin_1), U9.5 (M2A)
- new net: J4.4 (Pin_4), J7.4 (Pin_4), U9.6 (M2B)
- new net: D12.2 (A), R30.2
- new net: R45.2, R46.2, U13.9
- new net: D9.2 (A), R27.2
- new net: J2.A5 (CC1), R19.1
- new net: D4.1 (K), R38.2
- new net: J2.B5 (CC2), R18.1
- new net: J6.3 (Pin_3), U11.3 (M1B)
- new net: J6.1 (Pin_1), U11.4 (M1A)
- new net: J6.2 (Pin_2), U11.5 (M2A)
- new net: J6.4 (Pin_4), U11.6 (M2B)
- new net: J14.3 (Pin_3), U13.6
- new net: D4.2 (A), J10.2 (Pin_2)
- new net: J12.1 (Pin_1), R36.1
- new net: R36.2, U12.8
- new net: D2.1 (K), R5.1
- new net: R14.1, U12.14
- new net: R33.2, U12.2
- new net: J9.1 (Pin_1), R33.1
- new net: R10.1, SW2.1
- new net +3.3V: C1.1, C11.1, C12.1, C15.1, C16.1, C2.1, MICRO_SD1.4 (VDD), R11.1, R12.1, R15.1, R17.1, R23.1, R24.1, R25.1, R26.1, R32.1, R8.1, U1.2 (VDD), U10.2 (VIO), U11.2 (VIO), U3.2 (VO), U4.6 (VDD), U4.7 (VREGIN), U8.2 (VIO), U9.2 (VIO)
- new net +5V: C10.1, C19.1, C20.1, C22.1, C23.1, C24.1, C29.1, C8.1, C9.1, D2.2 (A), L1.2, R22.1, R3.1, U12.1, U12.3, U12.5, U12.7, U13.14 (VCC), U3.3 (VI), U6.16 (VCC), U7.16 (VCC)
- new net AHCT2: U6.9 (QH'), U7.14 (SER)
- new net A_CS: U11.13 (CS), U7.6 (QG)
- new net A_DIAG: R24.2, U1.4 (SENSOR_VP), U11.18 (DIAG1)
- new net A_DIR: U11.9 (DIR), U7.4 (QE)
- new net A_EN: U11.16 (~{EN}), U7.7 (QH)
- new net A_SETP: R30.1, U11.10 (STEP)
- new net A_STEP: U7.5 (QF)
- new net DTR: Q1.4 (E2), R6.1, U4.28 (~{DTR})
- new net ESP_EN: C13.1, Q1.6 (C1), R8.2, SW1.2, U1.3 (EN)
- new net GND: C1.2, C10.2, C11.2, C12.2, C13.2, C14.2, C15.2, C16.2, C17.2, C18.2, C19.2, C2.2, C20.2, C21.2, C22.2, C23.2, C24.2, C25.2, C26.2, C27.2, C28.2, C29.2, C3.2, C4.2, C6.2, C7.2, C8.2, C9.2, D1.A, D10.1 (K), D11.1 (K), D12.1 (K), D9.1 (K), J1.1 (Pin_1), J13.2 (Pin_2), J14.2 (Pin_2), J15.2 (Pin_2), J16.2 (Pin_2), J2.A1 (GND), J2.A12 (GND), J2.B1 (GND), J2.B12 (GND), J2.S1 (SHIELD), MICRO_SD1.6 (VSS), MICRO_SD1.MP1 (SHIELD), MICRO_SD1.MP2 (SHIELD), MICRO_SD1.MP3 (SHIELD), MICRO_SD1.MP4 (SHIELD), R1.2, R10.2, R18.2, R19.2, R20.2, R21.2, R37.1, R38.1, R39.1, R4.2, R40.1, R42.1, R44.1, R46.1, R48.1, R5.2, R9.2, SW1.SH (B), SW2.SH (B), U1.1 (GND), U1.15 (GND), U1.38 (GND), U1.39 (GND), U10.1 (GND), U10.7 (GND), U11.1 (GND), U11.7 (GND), U12.11, U12.13, U12.15, U12.9, U13.1, U13.10, U13.13, U13.4, U13.7 (GND), U2.7 (GND), U2.9 (GNDPAD), U3.1 (GND), U4.29 (GND), U4.3 (GND), U5.3, U6.13 (~{OE}), U6.8 (GND), U7.13 (~{OE}), U7.8 (GND), U8.1 (GND), U8.7 (GND), U9.1 (GND), U9.7 (GND)
- new net GPIO0: C14.1, Q1.3 (C2), R11.2, SW2.2
- new net GPIO25: U1.10 (IO25)
- new net GPIO26: U1.11 (IO26)
- new net GPIO27: U1.12 (IO27)
- new net GPIO32: U1.8 (IO32)
- new net GPIO33: U1.9 (IO33)
- new net I2S_BCK: R20.1, R21.1, U1.36 (IO22), U6.11 (SRCLK), U7.11 (SRCLK)
- new net I2S_DATA: U1.33 (IO21), U6.14 (SER)
- new net I2S_MR: C21.1, R22.2, U6.10 (~{SRCLR}), U7.10 (~{SRCLR})
- new net I2S_WS: U1.28 (IO17), U6.12 (RCLK), U7.12 (RCLK)
- new net IN_1: R12.2, R13.2, U1.25 (IO0)
- new net IN_2: R14.2, R15.2, U1.24 (IO2)
- new net IN_3: R16.2, R17.2, U1.26 (IO4)
- new net IN_4: R31.2, R32.2, U1.14 (IO12)
- new net MISO: MICRO_SD1.7 (DAT0), U1.31 (IO19), U10.12 (SDO), U11.12 (SDO), U8.12 (SDO), U9.12 (SDO)
- new net MOSI: MICRO_SD1.3 (CMD), U1.37 (IO23), U10.15 (SDI), U11.15 (SDI), U8.15 (SDI), U9.15 (SDI)
- new net PWM_1: R41.1, U1.16 (IO13)
- new net PWM_2: R43.1, U1.13 (IO14)
- new net PWM_3: R45.1, U1.23 (IO15)
- new net PWM_4: R47.1, U1.27 (IO16)
- new net RST: Q1.1 (E1), R7.1, U4.24 (~{RTS})
- new net RX0: U1.34 (RXD0/IO3), U4.25 (RXD)
- new net SCK: MICRO_SD1.5 (CLK), U1.30 (IO18), U10.14 (SCK), U11.14 (SCK), U8.14 (SCK), U9.14 (SCK)
- new net SD_CS: MICRO_SD1.2 (CD/DAT3), U1.29 (IO5)
- new net TX0: U1.35 (TXD0/IO1), U4.26 (TXD)
- new net VBUS: C17.1, C18.1, J2.A4 (VBUS), J2.A9 (VBUS), J2.B4 (VBUS), J2.B9 (VBUS), U4.8 (VBUS), U5.5
- new net VDC: C25.1, C26.1, C27.1, C28.1, C3.1, C4.1, J1.2 (Pin_2), J13.1 (Pin_1), J14.1 (Pin_1), J15.1 (Pin_1), J16.1 (Pin_1), U10.8 (VM), U11.8 (VM), U2.2 (VIN), U8.8 (VM), U9.8 (VM)
- new net X_CS: U6.3 (QD), U8.13 (CS)
- new net X_DIAG: R26.2, U1.6 (IO34), U8.18 (DIAG1)
- new net X_DIR: U6.1 (QB), U8.9 (DIR)
- new net X_EN: U6.15 (QA), U8.16 (~{EN})
- new net X_SETP: R27.1, U6.2 (QC), U8.10 (STEP)
- new net Y_CS: U6.6 (QG), U9.13 (CS)
- new net Y_DIAG: R25.2, U1.7 (IO35), U9.18 (DIAG1)
- new net Y_DIR: U6.4 (QE), U9.9 (DIR)
- new net Y_EN: U6.7 (QH), U9.16 (~{EN})
- new net Y_SETP: R28.1, U9.10 (STEP)
- new net Y_STEP: U6.5 (QF)
- new net Z_CS: U10.13 (CS), U7.3 (QD)
- new net Z_DIAG: R23.2, U1.5 (SENSOR_VN), U10.18 (DIAG1)
- new net Z_DIR: U10.9 (DIR), U7.1 (QB)
- new net Z_EN: U10.16 (~{EN}), U7.15 (QA)
- new net Z_SETP: R29.1, U10.10 (STEP)
- new net Z_STEP: U7.2 (QC)
- no-connect marks 0 -> 30

Commit message: schematics ready
Parts:
- added D13, D15: LED, symbol Device:LED
- added D14, D16: B340, Diode_SMD:D_SMC, symbol Diode:B340
- added D7, D8: B340, Diode_SMD:D_SMB-SMC_Universal_Handsoldering, symbol Diode:B340
- added J17, J18: Conn_01x03_Pin, Connector_JST:JST_PH_B3B-PH-K_1x03_P2.00mm_Vertical, symbol Connector:Conn_01x03_Pin
- added J19, J20: Conn_01x02_Pin, symbol Connector:Conn_01x02_Pin
- added K1, K2: Relay_SPDT, Relay_THT:Relay_SPDT_Omron-G5Q-1, symbol Relay:Relay_SPDT
- added Q2, Q3: PMBT3904YS, Package_TO_SOT_SMD:SOT-363_SC-70-6_Handsoldering, symbol Transistor_BJT:PMBT3904YS
- added Q4: FDS4559, Package_TO_SOT_SMD:SOT-223-3_TabPin2, symbol Transistor_FET:FDS4559
- added R49, R50: 1k, Resistor_SMD:R_0805_2012Metric_Pad1.20x1.40mm_HandSolder, symbol Device:R
- added R51, R52, R53, R54: R, Resistor_SMD:R_0805_2012Metric_Pad1.20x1.40mm_HandSolder, symbol Device:R
Connections:
- net +5V: now also D7.1 (K), D8.1 (K), K1.A1, K2.A1
- net GND: now also D13.1 (K), D15.1 (K), Q2.4 (E2), Q3.4 (E2), Q4.1 (S1), Q4.3 (S2)
- net VDC: now also D14.1 (K), D16.1 (K), J19.2 (Pin_2), J20.2 (Pin_2)
- net GPIO26 renamed SW2
- net SW2: now also R53.1, R54.1
- net GPIO27 renamed SW1
- net SW1: now also R51.1, R52.1
- net GPIO32 renamed RELAY2
- net RELAY2: now also R50.1
- net GPIO33 renamed RELAY1
- net RELAY1: now also R49.1
- new net: J17.2 (Pin_2), K1.11
- new net: J17.1 (Pin_1), K1.12
- new net: J17.3 (Pin_3), K1.14
- new net: D7.2 (A), K1.A2, Q2.3 (C2)
- new net: Q2.5 (B2), R49.2
- new net: D15.2 (A), R53.2
- new net: Q4.4 (G2), R54.2
- new net: D16.2 (A), J20.1 (Pin_1), Q4.5 (D2), Q4.6 (D2)
- new net: J18.2 (Pin_2), K2.11
- new net: J18.1 (Pin_1), K2.12
- new net: J18.3 (Pin_3), K2.14
- new net: D8.2 (A), K2.A2, Q3.3 (C2)
- new net: D13.2 (A), R51.2
- new net: Q4.2 (G1), R52.2
- new net: D14.2 (A), J19.1 (Pin_1), Q4.7 (D1), Q4.8 (D1)
- new net: Q3.5 (B2), R50.2

Commit message: board preparation
Parts:
- D13, D15: footprint (none) -> LED_SMD:LED_0805_2012Metric_Pad1.15x1.40mm_HandSolder
- J19, J20: footprint (none) -> Connector_JST:JST_PH_B2B-PH-K_1x02_P2.00mm_Vertical
Changed lines of the file:
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@@
 			)
 		)
-		(property "Footprint" ""
+		(property "Footprint" "LED_SMD:LED_0805_2012Metric_Pad1.15x1.40mm_HandSolder"
 			(at 416.56 237.49 0)
 			(effects
@@
 			)
 		)
-		(property "Footprint" ""
+		(property "Footprint" "Connector_JST:JST_PH_B2B-PH-K_1x02_P2.00mm_Vertical"
 			(at 467.36 209.55 0)
 			(effects
@@
 			)
 		)
-		(property "Footprint" ""
+		(property "Footprint" "Connector_JST:JST_PH_B2B-PH-K_1x02_P2.00mm_Vertical"
 			(at 453.39 261.62 0)
 			(effects
@@
 			)
 		)
-		(property "Footprint" ""
+		(property "Footprint" "LED_SMD:LED_0805_2012Metric_Pad1.15x1.40mm_HandSolder"
 			(at 402.59 289.56 0)
 			(effects
